Commit message: change to dae

File: thesis/urdf/lf064.urdf.xacro (robot description, xacro)
@@ -27,5 +27,5 @@
         <origin rpy="0 0 0" xyz="0 0 0" />
         <geometry>
-          <mesh filename="file://$(arg modelDir)/meshes/lf064-$(arg modelNr).stl" scale="$(arg scale)"/>
+          <mesh filename="file://$(arg modelDir)/meshes/lf064-$(arg modelNr).dae" scale="$(arg scale)"/>
         </geometry>
         <material name="grey">
@@ -36,5 +36,5 @@
         <origin rpy="0 0 0" xyz="0 0 0" />
           <geometry>
-            <mesh filename="file://$(arg modelDir)/meshes/lf064-$(arg modelNr).stl" scale="$(arg scale)"/>
+            <mesh filename="file://$(arg modelDir)/meshes/lf064-$(arg modelNr).dae" scale="$(arg scale)"/>
             <!--box size="0.8 0.8 1"/-->
            </geometry>
