Commit message: update urdf inertial info

File: thesis/urdf/lf06401.urdf.xacro (robot description, xacro)
@@ -17,7 +17,7 @@
     <link name="link_lf06401">
       <inertial>
-        <mass value="5"/>
-          <origin xyz="0 0 0.6"/>
-            <inertia  ixx="5.0" ixy="0.0"  ixz="0.0"  iyy="5.0"  iyz="0.0"  izz="5.0" />
+        <mass value="0.242"/>
+          <origin xyz="0 0.000497 0.0"/>
+            <inertia  ixx="0.0003335" ixy="0.0"  ixz="0.0"  iyy="0.0001565"  iyz="0.0"  izz="0.0004809" />
       </inertial>
      <visual>

File: thesis/urdf/lf06402.urdf.xacro (robot description, xacro)
@@ -17,7 +17,7 @@
     <link name="link_lf06402">
       <inertial>
-        <mass value="0.5"/>
-          <origin xyz="0 0 0"/>
-            <inertia  ixx="1.0" ixy="0.0"  ixz="0.0"  iyy="1.0"  iyz="0.0"  izz="1.0" />
+        <mass value="0.00796"/>
+          <origin xyz="0 0 0.018"/>
+            <inertia  ixx="0.000000716" ixy="0.0"  ixz="0.0"  iyy="0.000000716"  iyz="0.0"  izz="0.0000001144" />
       </inertial>
      <visual>

File: thesis/urdf/lf06403.urdf.xacro (robot description, xacro)
@@ -17,7 +17,7 @@
     <link name="link_lf06403">
       <inertial>
-        <mass value="1"/>
-          <origin xyz="0 0 0"/>
-            <inertia  ixx="2.0" ixy="0.0"  ixz="0.0"  iyy="2.0"  iyz="0.0"  izz="2.0" />
+        <mass value="0.0809"/>
+          <origin xyz="0 0.009644 0"/>
+            <inertia  ixx="0.00004879" ixy="0.0"  ixz="0.0"  iyy="0.00007025"  iyz="0.0"  izz="0.00007138" />
       </inertial>
      <visual>

File: thesis/urdf/lf06404.urdf.xacro (robot description, xacro)
@@ -17,7 +17,7 @@
     <link name="link_lf06404">
       <inertial>
-        <mass value="0.8"/>
-          <origin xyz="0 0 0"/>
-            <inertia  ixx="1.0" ixy="0.0"  ixz="0.0"  iyy="1.0"  iyz="0.0"  izz="1.0" />
+        <mass value="0.0187"/>
+          <origin xyz="0 0 0.01775"/>
+            <inertia  ixx="0.000001897" ixy="0.0"  ixz="0.0"  iyy="0.000001897"  iyz="0.0"  izz="0.0000006385" />
       </inertial>
      <visual>

File: thesis/urdf/lf06405.urdf.xacro (robot description, xacro)
@@ -17,7 +17,7 @@
     <link name="link_lf06405">
       <inertial>
-        <mass value="1.5"/>
-          <origin xyz="0 0 0"/>
-            <inertia  ixx="1.0" ixy="0.0"  ixz="0.0"  iyy="1.0"  iyz="0.0"  izz="1.0" />
+        <mass value="0.043"/>
+          <origin xyz="0.022 0 0.00775"/>
+            <inertia  ixx="0.000002604" ixy="0.0"  ixz="0.0"  iyy="0.00002338"  iyz="0.0"  izz="0.00002423" />
       </inertial>
      <visual>
