Commit message: add gripperHwInterface arg in lauch,xacro; fix rviz movegroup model

File: thesis/urdf/iiwa7_integration.urdf.xacro (robot description, xacro)
@@ -10,8 +10,9 @@
   <xacro:include filename="$(find thesis)/urdf/add_table.xacro" />
   <xacro:arg name="hardware_interface" default="PositionJointInterface"/>
+  <xacro:arg name="gripperHwInterface" default="EffortJointInterface"/>
   <xacro:arg name="robot_name" default="iiwa"/>
   <xacro:arg name="table_origin_xyz" default="0 0 1.2"/>
   <xacro:arg name="table_origin_rpy" default="0 0 0"/>
-  <xacro:arg name="origin_xyz" default="0 0 0"/>
+  <xacro:arg name="origin_xyz" default="0 -0.3 0"/>
   <xacro:arg name="origin_rpy" default="0 0 0"/>
   <xacro:arg name="table_ee" default="table_ee"/>
@@ -27,5 +28,5 @@
   </xacro:iiwa7>
   <!-- schunk greifer  -->
-  <xacro:wsg_50_xacro name="wsg50" parent="iiwa_link_ee">
+  <xacro:wsg_50_xacro name="wsg50" parent="iiwa_link_ee" gripperHwInterface="$(arg gripperHwInterface)">
     <origin xyz="0 0 0.01" rpy= "0 0 0"/>
   </xacro:wsg_50_xacro>

File: wsg50-ros-pkg/wsg_50_simulation/urdf/wsg_50.urdf.xacro (robot description, xacro)
@@ -8,5 +8,5 @@
 <!-- finger_tip:    Offset of finger tip along fingers' motion direction.
                     Use e.g. for single contact point tip on finger. (default 0) -->
-<xacro:macro name="wsg_50_xacro" params="name parent *origin">
+<xacro:macro name="wsg_50_xacro" params="name parent gripperHwInterface *origin">
  <joint name="${name}_anterior_gripper_joint" type="fixed">
     <xacro:insert_block name="origin"/>
@@ -59,12 +59,10 @@
      <type>transmission_interface/SimpleTransmission</type>
      <actuator name="${name}_base_motor_left">
-       <!--hardwareInterface>hardware_interface/EffortJointInterface</hardwareInterface-->
-       <hardwareInterface>hardware_interface/PositionJointInterface</hardwareInterface>
+       <hardwareInterface>hardware_interface/${gripperHwInterface}</hardwareInterface>
        <mechanicalReduction>1</mechanicalReduction>
        <!--motorTorqueConstant>1</motorTorqueConstant-->
      </actuator>
      <joint name="${name}_gripper_left_joint">
-       <!--hardwareInterface>hardware_interface/EffortJointInterface</hardwareInterface-->
-       <hardwareInterface>hardware_interface/PositionJointInterface</hardwareInterface>
+      <hardwareInterface>hardware_interface/${gripperHwInterface}</hardwareInterface>
      </joint>
   </transmission>
@@ -113,12 +111,10 @@
      <type>transmission_interface/SimpleTransmission</type>
      <actuator name="${name}_base_motor_right">
-       <!--hardwareInterface>hardware_interface/EffortJointInterface</hardwareInterface-->
-       <hardwareInterface>hardware_interface/PositionJointInterface</hardwareInterface>
-       <mechanicalReduction>1</mechanicalReduction>
+        <hardwareInterface>hardware_interface/${gripperHwInterface}</hardwareInterface>
+        <mechanicalReduction>1</mechanicalReduction>
        <!--motorTorqueConstant>1</motorTorqueConstant-->
      </actuator>
      <joint name="${name}_gripper_right_joint">
-       <!--hardwareInterface>hardware_interface/EffortJointInterface</hardwareInterface-->
-       <hardwareInterface>hardware_interface/PositionJointInterface</hardwareInterface>
+        <hardwareInterface>hardware_interface/${gripperHwInterface}</hardwareInterface>
      </joint>
   </transmission>
@@ -154,10 +150,10 @@
     <turnGravityOff>false</turnGravityOff>
   </gazebo>
-<!--gazebo>
+<gazebo>
   <plugin name="gazebo_ros_control" filename="libgazebo_ros_control.so">
     <robotNamespace>/</robotNamespace>
   </plugin>
-</gazebo-->
-  <!--gazebo>
+</gazebo>
+  <gazebo>
     <controller:gazebo_ros_controller_manager name="gazebo_ros_controller_manager" plugin="libgazebo_ros_controller_manager.so">
       <alwaysOn>true</alwaysOn>
@@ -165,5 +161,5 @@
       <interface:audio name="gazebo_ros_controller_manager_dummy_iface" />
     </controller:gazebo_ros_controller_manager>
-  </gazebo-->
+  </gazebo>
 </xacro:macro>
 </robot>

File: wsg50-ros-pkg/wsg_50_simulation/urdf/wsg_test.xacro (robot description, xacro)
@@ -3,5 +3,6 @@
   <link name="footprint" />
   <xacro:include filename="$(find wsg_50_simulation)/urdf/wsg_50.urdf.xacro" />
-  <xacro:wsg_50_xacro name="wsg50" parent="footprint">
+  <xacro:wsg_50_xacro name="wsg50" parent="footprint" gripperHwInterface="EffortJointInterface">
+  <!-- <xacro:wsg_50_xacro name="wsg50" parent="footprint" gripperHwInterface="PositionJointInterface"> -->
     <pose xyz="0 0 0.05" rpy= "0 0 0"/>
   </xacro:wsg_50_xacro>

Commit message: update for ros-noetic,prepare for merging repo

File: thesis/urdf/iiwa7_integration.urdf.xacro (robot description, xacro)
@@ -17,5 +17,5 @@
   <xacro:arg name="origin_rpy" default="0 0 0"/>
   <xacro:arg name="table_ee" default="table_ee"/>
-  <xacro:arg name="modelDir" default="/root/exchange/tempData"/>
+  <xacro:arg name="modelDir" default="/root/exchange/tempData' )"/>
   <!-- Fix to world just for testing -->
   <link name="world"/>

File: thesis/urdf/lf064.urdf.xacro (robot description, xacro)
@@ -4,5 +4,5 @@
   <xacro:arg name="origin_rpy" default="'0 0 0'"/>
   <xacro:arg name="root_linkName" default="world"/>
-  <xacro:arg name="modelDir" default="/root/exchange/tempData"/>
+  <xacro:arg name="modelDir" default="$eval( env('HOME') + '/exchange/tempData')"/>
   <xacro:arg name="modelNr" default="01"/>
   <xacro:arg name="scale" default="'0.001 0.001 0.001'"/>

File: thesis/urdf/lf06401.urdf (robot description, URDF)
Before this commit: robot lf064, 2 links, 1 joints
Links:
- link link_lf06401: geometry collision mesh filename=file:///home/ubuntu/exchange/tempData/meshes/lf064-01.dae scale=0.001 0.001 0.001; visual mesh filename=file:///home/ubuntu/exchange/tempData/meshes/lf064-01.dae scale=0.001 0.001 0.001

File: thesis/urdf/lf06401.urdf.xacro (robot description, xacro)
@@ -4,5 +4,5 @@
   <xacro:arg name="origin_rpy" default="'0 0 0'"/>
   <xacro:arg name="root_linkName" default="world"/>
-  <xacro:arg name="modelDir" default="/root/exchange/tempData"/>
+  <xacro:arg name="modelDir" default="$eval( env('HOME') + '/exchange/tempData')"/>
   <xacro:arg name="scale" default="'0.001 0.001 0.001'"/>
   <xacro:include filename="$(find iiwa_description)/urdf/materials.xacro" />

File: thesis/urdf/lf06402.urdf (robot description, URDF)
Before this commit: robot lf064, 2 links, 1 joints
Links:
- link link_lf06402: geometry collision mesh filename=file:///home/ubuntu/exchange/tempData/meshes/lf064-02.dae scale=0.001 0.001 0.001; visual mesh filename=file:///home/ubuntu/exchange/tempData/meshes/lf064-02.dae scale=0.001 0.001 0.001

File: thesis/urdf/lf06402.urdf.xacro (robot description, xacro)
@@ -4,5 +4,5 @@
   <xacro:arg name="origin_rpy" default="'0 0 0'"/>
   <xacro:arg name="root_linkName" default="world"/>
-  <xacro:arg name="modelDir" default="/root/exchange/tempData"/>
+  <xacro:arg name="modelDir" default="$eval( env('HOME') + '/exchange/tempData')"/>
   <xacro:arg name="scale" default="'0.001 0.001 0.001'"/>
   <xacro:include filename="$(find iiwa_description)/urdf/materials.xacro" />

File: thesis/urdf/lf06403.urdf (robot description, URDF)
Before this commit: robot lf064, 2 links, 1 joints
Links:
- link link_lf06403: geometry collision mesh filename=file:///home/ubuntu/exchange/tempData/meshes/lf064-03.dae scale=0.001 0.001 0.001; visual mesh filename=file:///home/ubuntu/exchange/tempData/meshes/lf064-03.dae scale=0.001 0.001 0.001

File: thesis/urdf/lf06403.urdf.xacro (robot description, xacro)
@@ -4,5 +4,5 @@
   <xacro:arg name="origin_rpy" default="'0 0 0'"/>
   <xacro:arg name="root_linkName" default="world"/>
-  <xacro:arg name="modelDir" default="/root/exchange/tempData"/>
+  <xacro:arg name="modelDir" default="$eval( env('HOME') + '/exchange/tempData')"/>
   <xacro:arg name="scale" default="'0.001 0.001 0.001'"/>
   <xacro:include filename="$(find iiwa_description)/urdf/materials.xacro" />

File: thesis/urdf/lf06404.urdf (robot description, URDF)
Before this commit: robot lf064, 2 links, 1 joints
Links:
- link link_lf06404: geometry collision mesh filename=file:///home/ubuntu/exchange/tempData/meshes/lf064-04.dae scale=0.001 0.001 0.001; visual mesh filename=file:///home/ubuntu/exchange/tempData/meshes/lf064-04.dae scale=0.001 0.001 0.001

File: thesis/urdf/lf06404.urdf.xacro (robot description, xacro)
@@ -4,5 +4,5 @@
   <xacro:arg name="origin_rpy" default="'0 0 0'"/>
   <xacro:arg name="root_linkName" default="world"/>
-  <xacro:arg name="modelDir" default="/root/exchange/tempData"/>
+  <xacro:arg name="modelDir" default="$eval( env('HOME') + '/exchange/tempData')"/>
   <xacro:arg name="scale" default="'0.001 0.001 0.001'"/>
   <xacro:include filename="$(find iiwa_description)/urdf/materials.xacro" />

File: thesis/urdf/lf06405.urdf (robot description, URDF)
Before this commit: robot lf064, 2 links, 1 joints
Links:
- link link_lf06405: geometry collision mesh filename=file:///home/ubuntu/exchange/tempData/meshes/lf064-05.dae scale=0.001 0.001 0.001; visual mesh filename=file:///home/ubuntu/exchange/tempData/meshes/lf064-05.dae scale=0.001 0.001 0.001

File: thesis/urdf/lf06405.urdf.xacro (robot description, xacro)
@@ -4,5 +4,5 @@
   <xacro:arg name="origin_rpy" default="'0 0 0'"/>
   <xacro:arg name="root_linkName" default="world"/>
-  <xacro:arg name="modelDir" default="/root/exchange/tempData"/>
+  <xacro:arg name="modelDir" default="$eval( env('HOME') + '/exchange/tempData')"/>
   <xacro:arg name="scale" default="'0.001 0.001 0.001'"/>
   <xacro:include filename="$(find iiwa_description)/urdf/materials.xacro" />
