Commit message: rollback to python2

File: thesis/urdf/lf06401.urdf (robot description, URDF)
Before this commit: robot lf064, 2 links, 1 joints
Links:
- link link_lf06401: geometry collision mesh filename=file:///root/exchange/tempData/meshes/lf064-01.dae scale=0.001 0.001 0.001; visual mesh filename=file:///root/exchange/tempData/meshes/lf064-01.dae scale=0.001 0.001 0.001

File: thesis/urdf/lf06402.urdf (robot description, URDF)
Before this commit: robot lf064, 2 links, 1 joints
Links:
- link link_lf06402: geometry collision mesh filename=file:///root/exchange/tempData/meshes/lf064-02.dae scale=0.001 0.001 0.001; visual mesh filename=file:///root/exchange/tempData/meshes/lf064-02.dae scale=0.001 0.001 0.001

File: thesis/urdf/lf06403.urdf (robot description, URDF)
Before this commit: robot lf064, 2 links, 1 joints
Links:
- link link_lf06403: geometry collision mesh filename=file:///root/exchange/tempData/meshes/lf064-03.dae scale=0.001 0.001 0.001; visual mesh filename=file:///root/exchange/tempData/meshes/lf064-03.dae scale=0.001 0.001 0.001

File: thesis/urdf/lf06404.urdf (robot description, URDF)
Before this commit: robot lf064, 2 links, 1 joints
Links:
- link link_lf06404: geometry collision mesh filename=file:///root/exchange/tempData/meshes/lf064-04.dae scale=0.001 0.001 0.001; visual mesh filename=file:///root/exchange/tempData/meshes/lf064-04.dae scale=0.001 0.001 0.001

File: thesis/urdf/lf06405.urdf (robot description, URDF)
Before this commit: robot lf064, 2 links, 1 joints
Links:
- link link_lf06405: geometry collision mesh filename=file:///root/exchange/tempData/meshes/lf064-05.dae scale=0.001 0.001 0.001; visual mesh filename=file:///root/exchange/tempData/meshes/lf064-05.dae scale=0.001 0.001 0.001
