Commit message: fix gazebo error due to variablizae modelDir

File: thesis/urdf/add_table.xacro (robot description, xacro)
@@ -5,5 +5,5 @@
         xmlns:xacro="http://www.ros.org/wiki/xacro"
         name="add_table">
-  <xacro:macro name="add_table" params="table_ee parent *origin">
+  <xacro:macro name="add_table" params="table_ee modelDir parent *origin">
     <joint name="world2table_joint" type="fixed">
       <xacro:insert_block name="origin"/>>
@@ -22,5 +22,5 @@
         <!--origin rpy="0 0 0" xyz="0.0 0 -${0.99613/2}"/-->
         <geometry>
-          <mesh filename="package://thesis/meshes/lf064_base.stl" scale="0.001 0.001 0.001"/>
+          <mesh filename="file://${modelDir}/meshes/lf064_base.stl" scale="0.001 0.001 0.001"/>
           <!--box size="0.985 0.698 0.99613"/-->
         </geometry>
@@ -59,5 +59,5 @@
         <origin rpy="0 0 0" xyz="0.0 0 0"/>
         <geometry>
-          <mesh filename="package://thesis/meshes/lf064_table.stl" scale="0.001 0.001 0.001"/>
+          <mesh filename="file://${modelDir}/meshes/lf064_table.stl" scale="0.001 0.001 0.001"/>
         <!--box size="0.146 0.05 0.0735"/-->
         </geometry>
@@ -69,5 +69,5 @@
         <origin rpy="0 0 0" xyz="0.0 0 0"/>
           <geometry>
-            <mesh filename="package://thesis/meshes/lf064_table.stl" scale="0.001 0.001 0.001"/>
+            <mesh filename="file://${modelDir}/meshes/lf064_table.stl" scale="0.001 0.001 0.001"/>
           </geometry>
       </collision>

File: thesis/urdf/iiwa7_integration.urdf.xacro (robot description, xacro)
@@ -16,7 +16,8 @@
   <xacro:arg name="origin_rpy" default="0 0 0"/>
   <xacro:arg name="table_ee" default="table_ee"/>
+  <xacro:arg name="modelDir" default="/root/exchange/tempData"/>
   <!-- Fix to world just for testing -->
   <link name="world"/>
-  <xacro:add_table table_ee="$(arg table_ee)"  parent="world">
+  <xacro:add_table table_ee="$(arg table_ee)" modelDir="$(arg modelDir)"  parent="world">
     <origin xyz="$(arg table_origin_xyz)" rpy="$(arg table_origin_rpy)" />
   </xacro:add_table>

File: thesis/urdf/lf064.urdf.xacro (robot description, xacro)
@@ -27,5 +27,5 @@
         <origin rpy="0 0 0" xyz="0 0 0" />
         <geometry>
-          <mesh filename="file://${modelDir}/meshes/lf064-$(arg modelNr).stl" scale="$(arg scale)"/>
+          <mesh filename="file://$(arg modelDir)/meshes/lf064-$(arg modelNr).stl" scale="$(arg scale)"/>
         </geometry>
         <material name="grey">
@@ -36,5 +36,5 @@
         <origin rpy="0 0 0" xyz="0 0 0" />
           <geometry>
-            <mesh filename="file://${modelDir}/meshes/lf064-$(arg modelNr).stl" scale="$(arg scale)"/>
+            <mesh filename="file://$(arg modelDir)/meshes/lf064-$(arg modelNr).stl" scale="$(arg scale)"/>
             <!--box size="0.8 0.8 1"/-->
            </geometry>

Commit message: newSetup for kinect2

File: thesis/urdf/add_table.xacro (robot description, xacro)
@@ -15,13 +15,13 @@
       <inertial>
         <mass value="80"/>
-          <origin xyz="0 0 -${0.997/2}" />
+          <origin xyz="0 0 -${0.5}" />
             <inertia  ixx="${80/12*(0.698*0.698+0.997*0.997)}" ixy="0.0"  ixz="0.0"  iyy="${80/12*(0.685*0.685+0.997*0.997)}"  iyz="0.0"  izz="${80/12*(0.698*0.698+0.685*0.685)}" />
       </inertial>
      <visual>
-        <origin rpy="0 0 0" xyz="0.0 0 0"/>
+        <origin rpy="0 0 0" xyz="0.0 0 -${1.2/2 + 0.0075}"/>
         <!--origin rpy="0 0 0" xyz="0.0 0 -${0.99613/2}"/-->
         <geometry>
-          <mesh filename="file://${modelDir}/meshes/lf064_base.stl" scale="0.001 0.001 0.001"/>
-          <!--box size="0.985 0.698 0.99613"/-->
+          <!--mesh filename="file://${modelDir}/meshes/lf064_base.stl" scale="0.001 0.001 0.001"/-->
+          <box size="0.985 0.698 1.2"/>
         </geometry>
         <material name="grey">
@@ -31,8 +31,8 @@
       <collision>
         <!--origin rpy="0 0 0" xyz="0.0 0 0"/-->
-        <origin rpy="0 0 0" xyz="0.0 0 -${0.997/2}"/>
+        <origin rpy="0 0 0" xyz="0.0 0 -${1.2/2}"/>
           <geometry>
             <!--mesh filename="package://thesis/meshes/lf064_base.stl" scale="0.001 0.001 0.001"/-->
-            <box size="0.985 0.698 0.997"/>
+            <box size="0.985 0.698 1.2"/>
           </geometry>
       </collision>

File: thesis/urdf/iiwa7_integration.urdf.xacro (robot description, xacro)
@@ -11,5 +11,5 @@
   <xacro:arg name="hardware_interface" default="PositionJointInterface"/>
   <xacro:arg name="robot_name" default="iiwa"/>
-  <xacro:arg name="table_origin_xyz" default="0 0 0.997"/>
+  <xacro:arg name="table_origin_xyz" default="0 0 1.2"/>
   <xacro:arg name="table_origin_rpy" default="0 0 0"/>
   <xacro:arg name="origin_xyz" default="0 0 0"/>
@@ -30,4 +30,4 @@
     <origin xyz="0 0 0.01" rpy= "0 0 0"/>
   </xacro:wsg_50_xacro>
-  <xacro:sensor_kinect prefix="/" name="kinect2" parent="iiwa_link_ee" cam_px="0.0" cam_py="0.03" cam_pz="0.04" cam_or="${PI/2}" cam_op="${-PI/2}" cam_oy="0" />
+  <xacro:sensor_kinect prefix="/" name="kinect2" parent="iiwa_link_ee" cam_px="0.0" cam_py="0.02" cam_pz="0.08" cam_or="${PI/2}" cam_op="${-PI/2}" cam_oy="0" />
 </robot>

Commit message: reduce box size to avoid collision with table plate

File: thesis/urdf/add_table.xacro (robot description, xacro)
@@ -34,5 +34,5 @@
           <geometry>
             <!--mesh filename="package://thesis/meshes/lf064_base.stl" scale="0.001 0.001 0.001"/-->
-            <box size="0.985 0.698 1.2"/>
+            <box size="0.985 0.698 1.1"/>
           </geometry>
       </collision>
