Commit message: change gripper finger model to dae

File: wsg50-ros-pkg/wsg_50_simulation/urdf/wsg_50.urdf.xacro (robot description, xacro)
@@ -78,5 +78,5 @@
           <origin xyz="0.0 0 0" rpy="0 0 0" />
           <geometry>
-             <mesh filename="package://wsg_50_simulation/meshes/GUIDE_WSG50_110.stl" scale="0.001 0.001 0.001"/>
+             <mesh filename="package://wsg_50_simulation/meshes/GUIDE_WSG50_110.dae" scale="0.001 0.001 0.001"/>
 	     <!--box size="0.0175 0.03 0.024"/-->
           </geometry>
@@ -89,5 +89,5 @@
           <geometry>
 	     <!--box size="0.0175 0.03 0.024"/-->
-             <mesh filename="package://wsg_50_simulation/meshes/GUIDE_WSG50_110.stl" scale="0.001 0.001 0.001"/>
+             <mesh filename="package://wsg_50_simulation/meshes/GUIDE_WSG50_110.dae" scale="0.001 0.001 0.001"/>
          </geometry>
      </collision>
@@ -130,5 +130,5 @@
           <origin xyz="0.0 0 0" rpy="0 0 0" />
           <geometry>
-             <mesh filename="package://wsg_50_simulation/meshes/GUIDE_WSG50_110.stl" scale="0.001 0.001 0.001"/>
+             <mesh filename="package://wsg_50_simulation/meshes/GUIDE_WSG50_110.dae" scale="0.001 0.001 0.001"/>
 	     <!--box size="0.0175 0.03 0.024"/-->
           </geometry>
@@ -141,5 +141,5 @@
           <geometry>
 	     <!--box size="0.0175 0.03 0.024"/-->
-             <mesh filename="package://wsg_50_simulation/meshes/GUIDE_WSG50_110.stl" scale="0.001 0.001 0.001"/>
+             <mesh filename="package://wsg_50_simulation/meshes/GUIDE_WSG50_110.dae" scale="0.001 0.001 0.001"/>
          </geometry>
      </collision>
