Commit message: change stl to dae

File: depth_sensors/kinect_description/urdf/kinect/kinect2.xacro (robot description, xacro)
@@ -24,5 +24,5 @@
             <visual>
                 <geometry>
-                    <mesh filename="package://kinect_description/meshes/sensors/kinect2.stl" scale="0.001 0.001 0.001"/>
+                    <mesh filename="package://kinect_description/meshes/sensors/kinect2.dae" scale="0.001 0.001 0.001"/>
                 </geometry>
                 <origin xyz="0 0 0" rpy="-1.57 0 -1.57"/>

Commit message: change orientation due to new kinect2 model

File: depth_sensors/kinect_description/urdf/kinect/kinect2.xacro (robot description, xacro)
@@ -26,5 +26,5 @@
                     <mesh filename="package://kinect_description/meshes/sensors/kinect2.dae" scale="0.001 0.001 0.001"/>
                 </geometry>
-                <origin xyz="0 0 0" rpy="-1.57 0 -1.57"/>
+                <origin xyz="0 0 0" rpy="0 0 $-{PI/2}"/>
                 <material name="black"/>
             </visual>

File: thesis/urdf/iiwa7_integration.urdf.xacro (robot description, xacro)
@@ -30,4 +30,4 @@
     <origin xyz="0 0 0.01" rpy= "0 0 0"/>
   </xacro:wsg_50_xacro>
-  <xacro:sensor_kinect prefix="/" name="kinect2" parent="iiwa_link_ee" cam_px="0.0" cam_py="0.03" cam_pz="0.075" cam_or="0" cam_op="0" cam_oy="0" />
+  <xacro:sensor_kinect prefix="/" name="kinect2" parent="iiwa_link_ee" cam_px="0.0" cam_py="0.03" cam_pz="0.075" cam_or="0" cam_op="0" cam_oy="${PI/2}" />
 </robot>

Commit message: try to fix coordinate assignment

File: depth_sensors/kinect_description/urdf/kinect/kinect2.xacro (robot description, xacro)
@@ -26,5 +26,5 @@
                     <mesh filename="package://kinect_description/meshes/sensors/kinect2.dae" scale="0.001 0.001 0.001"/>
                 </geometry>
-                <origin xyz="0 0 0" rpy="0 0 $-{PI/2}"/>
+                <origin xyz="0 0 0" rpy="1.57 0 -1.57"/>
                 <material name="black"/>
             </visual>

File: thesis/urdf/iiwa7_integration.urdf.xacro (robot description, xacro)
@@ -30,4 +30,4 @@
     <origin xyz="0 0 0.01" rpy= "0 0 0"/>
   </xacro:wsg_50_xacro>
-  <xacro:sensor_kinect prefix="/" name="kinect2" parent="iiwa_link_ee" cam_px="0.0" cam_py="0.03" cam_pz="0.075" cam_or="0" cam_op="0" cam_oy="${PI/2}" />
+  <xacro:sensor_kinect prefix="/" name="kinect2" parent="iiwa_link_ee" cam_px="0.0" cam_py="0.03" cam_pz="0.075" cam_or="-${PI/2}" cam_op="0" cam_oy="${PI/2}" />
 </robot>

Commit message: change orientation test

File: depth_sensors/kinect_description/urdf/kinect/kinect2.xacro (robot description, xacro)
@@ -26,5 +26,5 @@
                     <mesh filename="package://kinect_description/meshes/sensors/kinect2.dae" scale="0.001 0.001 0.001"/>
                 </geometry>
-                <origin xyz="0 0 0" rpy="1.57 0 -1.57"/>
+                <origin xyz="0 0 0" rpy="1.57 -1.57 0"/>
                 <material name="black"/>
             </visual>

File: thesis/urdf/iiwa7_integration.urdf.xacro (robot description, xacro)
@@ -30,4 +30,4 @@
     <origin xyz="0 0 0.01" rpy= "0 0 0"/>
   </xacro:wsg_50_xacro>
-  <xacro:sensor_kinect prefix="/" name="kinect2" parent="iiwa_link_ee" cam_px="0.0" cam_py="0.03" cam_pz="0.075" cam_or="-${PI/2}" cam_op="0" cam_oy="${PI/2}" />
+  <xacro:sensor_kinect prefix="/" name="kinect2" parent="iiwa_link_ee" cam_px="0.0" cam_py="0.03" cam_pz="0.075" cam_or="${PI/2}" cam_op="${-PI/2}" cam_oy="0" />
 </robot>

Commit message: try to fix wrong origin of dae

File: depth_sensors/kinect_description/urdf/kinect/kinect2.xacro (robot description, xacro)
@@ -26,5 +26,5 @@
                     <mesh filename="package://kinect_description/meshes/sensors/kinect2.dae" scale="0.001 0.001 0.001"/>
                 </geometry>
-                <origin xyz="0 0 0" rpy="1.57 -1.57 0"/>
+                <origin xyz="0 0 0" rpy="0 0 0"/>
                 <material name="black"/>
             </visual>

File: thesis/urdf/iiwa7_integration.urdf.xacro (robot description, xacro)
@@ -30,4 +30,4 @@
     <origin xyz="0 0 0.01" rpy= "0 0 0"/>
   </xacro:wsg_50_xacro>
-  <xacro:sensor_kinect prefix="/" name="kinect2" parent="iiwa_link_ee" cam_px="0.0" cam_py="0.03" cam_pz="0.075" cam_or="${PI/2}" cam_op="${-PI/2}" cam_oy="0" />
+  <xacro:sensor_kinect prefix="/" name="kinect2" parent="iiwa_link_ee" cam_px="0.0" cam_py="0.3" cam_pz="0.075" cam_or="${PI/2}" cam_op="${-PI/2}" cam_oy="0" />
 </robot>

Commit message: change orientation of kinect2.dae

File: depth_sensors/kinect_description/urdf/kinect/kinect2.xacro (robot description, xacro)
@@ -26,5 +26,5 @@
                     <mesh filename="package://kinect_description/meshes/sensors/kinect2.dae" scale="0.001 0.001 0.001"/>
                 </geometry>
-                <origin xyz="0 0 0" rpy="0 0 0"/>
+                <origin xyz="0 0 0" rpy="1.57 1.57 0"/>
                 <material name="black"/>
             </visual>

File: thesis/urdf/iiwa7_integration.urdf.xacro (robot description, xacro)
@@ -30,4 +30,4 @@
     <origin xyz="0 0 0.01" rpy= "0 0 0"/>
   </xacro:wsg_50_xacro>
-  <xacro:sensor_kinect prefix="/" name="kinect2" parent="iiwa_link_ee" cam_px="0.0" cam_py="0.3" cam_pz="0.075" cam_or="${PI/2}" cam_op="${-PI/2}" cam_oy="0" />
+  <xacro:sensor_kinect prefix="/" name="kinect2" parent="iiwa_link_ee" cam_px="0.0" cam_py="0.03" cam_pz="0.09" cam_or="${PI/2}" cam_op="${-PI/2}" cam_oy="0" />
 </robot>

Commit message: fixed orientation of model

File: depth_sensors/kinect_description/urdf/kinect/kinect2.xacro (robot description, xacro)
@@ -26,5 +26,5 @@
                     <mesh filename="package://kinect_description/meshes/sensors/kinect2.dae" scale="0.001 0.001 0.001"/>
                 </geometry>
-                <origin xyz="0 0 0" rpy="1.57 1.57 0"/>
+                <origin xyz="0 0 0" rpy="-1.57 0 -1.57"/>
                 <material name="black"/>
             </visual>
